File: circuit/bak/circuit.kicad_pcb (KiCad board)
At the start: 2 copper layers, 109.5 x 50.1 mm, 69 parts, among them J1 audio-jack, P1 USB_A, U1 MIC5219BM5_SOT23-5

Commit message: circuit finish
Parts:
- added P-GND1: CONN_01X02, Pin_Headers:Pin_Header_Straight_1x02, B.Cu at (115.1, 99.9)
- added P-VDD1: CONN_01X02, Pin_Headers:Pin_Header_Straight_1x02, B.Cu at (110.1, 100.0)
- added W1: TEST_1P, test-pad:test-pad, F.Cu at (168.1, 94.8)
- added W10: TEST_1P, test-pad:test-pad, F.Cu at (177.0, 58.2)
- added W11: TEST_1P, test-pad:test-pad, F.Cu at (204.8, 70.2)
- added W12: TEST_1P, test-pad:test-pad, F.Cu at (166.2, 74.8)
- added W13: TEST_1P, test-pad:test-pad, F.Cu at (175.8, 79.7)
- added W14: TEST_1P, test-pad:test-pad, F.Cu at (166.6, 91.4)
- added W2: TEST_1P, test-pad:test-pad, F.Cu at (118.4, 101.4)
- added W3: TEST_1P, test-pad:test-pad, F.Cu at (140.1, 67.5)
- added W4: TEST_1P, test-pad:test-pad, F.Cu at (131.9, 96.7)
- added W5: TEST_1P, test-pad:test-pad, F.Cu at (148.2, 97.7)
- added W6: TEST_1P, test-pad:test-pad, F.Cu at (146.4, 87.6)
- added W7: TEST_1P, test-pad:test-pad, F.Cu at (111.4, 95.8)
- added W8: TEST_1P, test-pad:test-pad, F.Cu at (140.2, 88.3)
- added W9: TEST_1P, test-pad:test-pad, F.Cu at (142.5, 95.2)
Routing:
- net GND: track 338.9 -> 351.1 mm
- net VDD: track 146.0 -> 155.7 mm
- net /CON_LAMP: track 61.9 -> 67.3 mm
- net +24V: track 41.1 -> 45.0 mm
- net +6V: track 17.2 -> 20.8 mm
- net /ADC_BATT: track 31.3 -> 34.7 mm
- net /IND_PV_WKUP: track 29.6 -> 32.9 mm
- net GNDPWR: track 62.1 -> 65.4 mm
- net +3V3: track 139.9 -> 143.1 mm
- net /ADC_LAMP: track 182.4 -> 185.7 mm
- net /ADC_USB: track 159.5 -> 162.7 mm
- net /CON_PV: track 48.8 -> 51.7 mm
- net +15V: track 188.7 -> 191.7 mm
- net /CON_USB: track 79.8 -> 82.1 mm
