File: circuit/circuit.kicad_pcb (KiCad board)
At the start: 2 copper layers, 109.5 x 50.1 mm, 85 parts, among them J1 audio-jack, P1 USB_A, U1 MIC5219BM5_SOT23-5

Commit message: circuit fabricated
Parts:
- added G***: UBLIK, ublik:LOGO, F.Cu at (119.2, 70.9)
Routing:
- net VDD: track 155.7 -> 156.3 mm
- net +3V3: track 143.1 -> 143.7 mm
Other:
- net class Default: clearance 0.2 -> 0.1; via_dia 0.6 -> 1; via_drill 0.4 -> 0.5
- rule trace_clearance: 0.2 -> 0.1
- board text added: "UBLIK"
- board text added: "v0.1"

Commit message: list components
Parts:
- C-VREG1, C-VREG2: value C -> 100n
Changed lines of the file:
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@@
     (links 166)
     (no_connects 0)
-    (area 97.974999 51.247809 209.665132 107.583333)
+    (area 97.974999 55.524999 208.125001 106.225001)
     (thickness 1.6)
     (drawings 6)
@@
       (effects (font (size 1 1) (thickness 0.15)))
     )
-    (fp_text value C (at 0 2.1 90) (layer F.Fab)
+    (fp_text value 100n (at 0 2.1 90) (layer F.Fab)
       (effects (font (size 1 1) (thickness 0.15)))
     )
@@
       (effects (font (size 1 1) (thickness 0.15)))
     )
-    (fp_text value C (at 0 2.1) (layer F.Fab)
-      (effects (font (size 1 1) (thickness 0.15)))
-    )
+    (fp_text value 100n (at 0 2.1) (layer F.Fab)
+      (effects (font (size 1 1) (thickness 0.15)))
+    )
