File: circuit/circuit.sch (KiCad schematic (older format))
At the start: 85 parts, among them J1 audio-jack, P1 USB_A, U1 MIC5219BM5_SOT23-5

Commit message: list components
Parts:
- C-VREG1, C-VREG2: value C -> 100n
Changed lines of the file:
@@
 P 4700 6950
 F 0 "C-VREG2" H 4725 7050 50  0000 L CNN
-F 1 "C" H 4725 6850 50  0000 L CNN
+F 1 "100n" H 4725 6850 50  0000 L CNN
 F 2 "Capacitors_SMD:C_0805_HandSoldering" H 4738 6800 50  0001 C CNN
 F 3 "" H 4700 6950 50  0000 C CNN
@@
 P 3700 7300
 F 0 "C-VREG1" H 3725 7400 50  0000 L CNN
-F 1 "C" H 3725 7200 50  0000 L CNN
+F 1 "100n" H 3725 7200 50  0000 L CNN
 F 2 "Capacitors_SMD:C_0805_HandSoldering" H 3738 7150 50  0001 C CNN
 F 3 "" H 3700 7300 50  0000 C CNN
