File: circuit_1/circuit.kicad_pcb (KiCad board)
At the start: 2 copper layers, 104.1 x 51.2 mm, 80 parts, among them J1 audio-jack, P1 USB_A, U1 MIC5219BM5_SOT23-5

Commit message: new design
Parts:
- added U2: 78TV_TO220V, linear:TO220V, B.Cu at (146.1, 85.2)
- D-LAMP2: value D -> D_Schottky
- moved D-LAMP2 3.95 mm to (146.3, 86.8)
Connections:
- TR-LAMP1 pad S: Net-(J1-Pad2) -> Net-(TR-LAMP1-PadS)
Routing:
- net Net-(TR-LAMP1-PadS): track 0.00 -> 8.05 mm
- net GND: track 383.4 -> 391.1 mm
- net /ADC_LAMP: track 107.0 -> 109.8 mm
- net Net-(J1-Pad2): track 10.5 -> 13.0 mm
