File: circuit_1/circuit.sch (KiCad schematic (older format))
At the start: 69 parts, among them J1 audio-jack, P1 USB_A, U1 MIC5219BM5_SOT23-5

Commit message: new design
Parts:
- removed D-LAMP2: D, Diodes_SMD:SMA_Handsoldering, symbol D
- added D-LAMP2: D_Schottky, Diodes_SMD:SMA_Handsoldering, symbol D_Schottky
- added U2: 78TV_TO220V, linear:TO220V, symbol 78TV_TO220V
Connections:
- net ADC_LAMP: now also D-LAMP2.2 (A)
- net GND: now also D-LAMP2.1 (K), U2.2 (GND)
- net at TR-LAMP1.S: now also U2.1 (VI); no longer J1.2 (V+)
- new net: J1.2 (V+), U2.3 (VO)
Other:
- moved on the sheet: J1
